File: pandalLight/pandaLight.brd (EAGLE design)
At the start: 160 x 100 mm, 112 parts, among them J1 PJ-037A, U13 TPD12S016PWR, U15 PMOD-2X6, U16 PMOD-2X6, U17 PLR135-T10, U18 PLT133-T10W, U20 TP10SQ, U21 TP10SQ, U22 PAN1322, U23 6SLX9TQG144, U4 FT2232HL, U5 93LC46BT-I/OT, U6 51, U7 51, U8 TPD12S016PWR, X1 USBUB-S, X2 HDMI_RECEPTICAL_A, X4 HDMI_RECEPTICAL_A, Y1 403, Y2 20Mhz

Commit message: Minor changes; Still looking for decent pin protection
Parts:
- added R4, R6: 200, pandaLight:0402
Connections:
- new net N$2: R2.2, R4.2, SV3.2
- new net N$3: R3.2, R6.2, SV3.3
- net LEDS_CLK: now also R6.1; no longer R3.2, SV3.3
- net LEDS_DATA: now also R4.1; no longer R2.2, SV3.2
Routing:
- net GND: track 76.4 -> 73.7 mm
- net LEDS_DATA: track 2.63 -> 0.00 mm
- net LEDS_CLK: track 2.63 -> 0.00 mm
Changed lines of the file:
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@@
 <element name="R2" library="pandaLight" package="0402" value="10k" x="31" y="94.3" rot="R270"/>
 <element name="R3" library="pandaLight" package="0402" value="10k" x="32.2" y="94.3" rot="R270"/>
+<element name="R4" library="pandaLight" package="0402" value="200" x="-102.8" y="-2.5"/>
+<element name="R6" library="pandaLight" package="0402" value="200" x="-102.8" y="-7.4"/>
 </elements>
 <signals>
@@
 <wire x1="56.325" y1="86.325" x2="56.3" y2="86.3" width="0.254" layer="16"/>
 <via x="56.3" y="86.3" extent="1-16" drill="0.3302"/>
-<wire x1="53.075" y1="87.5" x2="53.075" y2="84.825" width="0.254" layer="16"/>
 <wire x1="48.6" y1="88.85" x2="47.65" y2="88.85" width="0.254" layer="16"/>
 <wire x1="47.65" y1="88.85" x2="47.6" y2="88.8" width="0.254" layer="16"/>
@@
 <wire x1="60.5" y1="86.2" x2="60.6" y2="86.3" width="0.254" layer="1"/>
 <via x="60.6" y="86.3" extent="1-16" drill="0.3302"/>
-<wire x1="53.075" y1="84.825" x2="53.1" y2="84.8" width="0.254" layer="16"/>
 <wire x1="49.2" y1="86.35" x2="48.25" y2="86.35" width="0.254" layer="1"/>
 <via x="48.2" y="86.3" extent="1-16" drill="0.3302"/>
@@
 <signal name="LEDS_DATA">
 <contactref element="U23" pad="P6"/>
-<contactref element="SV3" pad="2"/>
-<contactref element="R2" pad="2"/>
-<wire x1="31" y1="93.65" x2="31" y2="91.97" width="0.1778" layer="1"/>
-<wire x1="31" y1="91.97" x2="30.33" y2="91.3" width="0.1778" layer="1"/>
-<wire x1="31" y1="91.97" x2="65.18" y2="65.05" width="0" layer="19" extent="1-1"/>
+<contactref element="R4" pad="1"/>
+<wire x1="-103.45" y1="-2.5" x2="65.18" y2="65.05" width="0" layer="19" extent="1-1"/>
 </signal>
 <signal name="LEDS_CLK">
-<contactref element="SV3" pad="3"/>
 <contactref element="U23" pad="P5"/>
-<contactref element="R3" pad="2"/>
-<wire x1="32.2" y1="93.65" x2="32.2" y2="91.97" width="0.1778" layer="1"/>
-<wire x1="32.2" y1="91.97" x2="32.87" y2="91.3" width="0.1778" layer="1"/>
-<wire x1="32.87" y1="91.3" x2="65.18" y2="64.55" width="0" layer="19" extent="1-1"/>
+<contactref element="R6" pad="1"/>
+<wire x1="-103.45" y1="-7.4" x2="65.18" y2="64.55" width="0" layer="19" extent="1-1"/>
 </signal>
 <signal name="FPGA_CLK20">
@@
 <wire x1="-55.88" y1="48.17" x2="52.83" y2="60.2" width="0" layer="19" extent="1-1"/>
 </signal>
+<signal name="N$2">
+<contactref element="R4" pad="2"/>
+<contactref element="SV3" pad="2"/>
+<contactref element="R2" pad="2"/>
+<wire x1="30.33" y1="91.3" x2="31" y2="93.65" width="0" layer="19" extent="1-1"/>
+<wire x1="-102.15" y1="-2.5" x2="30.33" y2="91.3" width="0" layer="19" extent="1-1"/>
+</signal>
+<signal name="N$3">
+<contactref element="SV3" pad="3"/>
+<contactref element="R6" pad="2"/>
+<contactref element="R3" pad="2"/>
+<wire x1="32.87" y1="91.3" x2="32.2" y2="93.65" width="0" layer="19" extent="1-1"/>
+<wire x1="-102.15" y1="-7.4" x2="32.87" y2="91.3" width="0" layer="19" extent="1-1"/>
+</signal>
 </signals>
